Commit message: Redesign workspace architecture: arm_core, arm_hardware_interface, arm_controllers, arm_firmware
Co-authored-by: S-T-C-05 <75141337+S-T-C-05@users.noreply.github.com>

File: src/arm_core/urdf/arm.xacro (robot description, xacro)
@@ -17,5 +17,5 @@
       <origin xyz="0 0 0" rpy="0 0 0" />
       <geometry>
-        <mesh filename="package://my_package/meshes/base_link.STL" />
+        <mesh filename="package://arm_core/meshes/base_link.STL" />
       </geometry>
       <material name="">
@@ -26,5 +26,5 @@
       <origin xyz="0 0 0" rpy="0 0 0" />
       <geometry>
-        <mesh filename="package://my_package/meshes/base_link.STL" />
+        <mesh filename="package://arm_core/meshes/base_link.STL" />
       </geometry>
     </collision>
@@ -46,5 +46,5 @@
       <origin xyz="0 0 0" rpy="0 0 0" />
       <geometry>
-        <mesh filename="package://my_package/meshes/bracket_link.STL" />
+        <mesh filename="package://arm_core/meshes/bracket_link.STL" />
       </geometry>
       <material name="">
@@ -55,5 +55,5 @@
       <origin xyz="0 0 0" rpy="0 0 0" />
       <geometry>
-        <mesh filename="package://my_package/meshes/bracket_link.STL" />
+        <mesh filename="package://arm_core/meshes/bracket_link.STL" />
       </geometry>
     </collision>
@@ -83,5 +83,5 @@
       <origin xyz="0 0 0" rpy="0 0 0" />
       <geometry>
-        <mesh filename="package://my_package/meshes/humerus_link.STL" />
+        <mesh filename="package://arm_core/meshes/humerus_link.STL" />
       </geometry>
       <material name="">
@@ -92,5 +92,5 @@
       <origin xyz="0 0 0" rpy="0 0 0" />
       <geometry>
-        <mesh filename="package://my_package/meshes/humerus_link.STL" />
+        <mesh filename="package://arm_core/meshes/humerus_link.STL" />
       </geometry>
     </collision>
@@ -120,5 +120,5 @@
       <origin xyz="0 0 0" rpy="0 0 0" />
       <geometry>
-        <mesh filename="package://my_package/meshes/forearm_link.STL" />
+        <mesh filename="package://arm_core/meshes/forearm_link.STL" />
       </geometry>
       <material name="">
@@ -129,5 +129,5 @@
       <origin xyz="0 0 0" rpy="0 0 0" />
       <geometry>
-        <mesh filename="package://my_package/meshes/forearm_link.STL" />
+        <mesh filename="package://arm_core/meshes/forearm_link.STL" />
       </geometry>
     </collision>
@@ -157,5 +157,5 @@
       <origin xyz="0 0 0" rpy="0 0 0" />
       <geometry>
-        <mesh filename="package://my_package/meshes/ubracket_link.STL" />
+        <mesh filename="package://arm_core/meshes/ubracket_link.STL" />
       </geometry>
       <material name="">
@@ -166,5 +166,5 @@
       <origin xyz="0 0 0" rpy="0 0 0" />
       <geometry>
-        <mesh filename="package://my_package/meshes/ubracket_link.STL" />
+        <mesh filename="package://arm_core/meshes/ubracket_link.STL" />
       </geometry>
     </collision>
@@ -194,5 +194,5 @@
       <origin xyz="0 0 0" rpy="0 0 0" />
       <geometry>
-        <mesh filename="package://my_package/meshes/endeffector_link.STL" />
+        <mesh filename="package://arm_core/meshes/endeffector_link.STL" />
       </geometry>
       <material name="">
@@ -203,5 +203,5 @@
       <origin xyz="0 0 0" rpy="0 0 0" />
       <geometry>
-        <mesh filename="package://my_package/meshes/endeffector_link.STL" />
+        <mesh filename="package://arm_core/meshes/endeffector_link.STL" />
       </geometry>
     </collision>

File: src/arm_moveit_config/config/arm_v3.urdf.xacro (robot description, xacro)
@@ -3,5 +3,5 @@
     <xacro:arg name="initial_positions_file" default="initial_positions.yaml" />
     <!-- Import arm_v3 urdf file -->
-    <xacro:include filename="$(find my_package)/urdf/arm.xacro" />
+    <xacro:include filename="$(find arm_core)/urdf/arm.xacro" />
     <!-- Import control_xacro -->
     <xacro:include filename="arm_v3.ros2_control.xacro" />
